File: Eagle/PiDriver/PiDriverV3/PiDriverV3.sch (EAGLE design)
At the start: 47 parts, among them IC1 L293E, IC2 L293E

Commit message: A second quote of smps for PiDrive was added
Parts:
- removed R4: 1k, rcl:R-US_M1206
- added D17: BZV55-C3V3, diode:ZENER-DIODESOD80C
- added IC3: (no value), linear:LM2596S
- added J1: DCJ0202, con-jack:DCJ0202
- R1: value (none) -> 1.5k
- R3: value 1k -> 2k
- R5, R6, R7, R8: value (none) -> 220
- renumbered LED1 to POWER
Connections:
- removed net N$25: C1.1, R2.2, R4.2, U$1.RA0/AN0
- net GND: now also D17.A, J1.3
- net N$28: now also C1.1, D17.C, R2.2, U$1.RA0/AN0; no longer R4.1
- net N$3: now also J1.1
Changed lines of the file:
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@@
 <part name="IC1" library="texas" deviceset="L293E" device=""/>
 <part name="IC2" library="texas" deviceset="L293E" device=""/>
-<part name="LED1" library="led" deviceset="LED" device="SMT1206"/>
-<part name="R1" library="rcl" deviceset="R-US_" device="M1206"/>
+<part name="POWER" library="led" deviceset="LED" device="SMT1206"/>
+<part name="R1" library="rcl" deviceset="R-US_" device="M1206" value="1.5k"/>
 <part name="S1" library="switch" deviceset="255SB" device=""/>
 <part name="LEFT" library="pinhead" deviceset="PINHD-1X2" device=""/>
@@
 <part name="U$1" library="SparkFun-DigitalIC" deviceset="PIC16F88-DIP" device=""/>
 <part name="R2" library="rcl" deviceset="R-US_" device="M1206" value="3.01k"/>
-<part name="R3" library="rcl" deviceset="R-US_" device="M1206" value="1k"/>
+<part name="R3" library="rcl" deviceset="R-US_" device="M1206" value="2k"/>
 <part name="C1" library="rcl" deviceset="C-US" device="C1206" value="10uF"/>
-<part name="R4" library="rcl" deviceset="R-US_" device="M1206" value="1k"/>
 <part name="RIGHTC" library="con-wago-508" deviceset="W237-02P" device=""/>
 <part name="LEFTC" library="con-wago-508" deviceset="W237-02P" device=""/>
@@
 <part name="AMRC" library="con-wago-508" deviceset="W237-02P" device=""/>
 <part name="LED2" library="led" deviceset="LED" device="SMT1206"/>
-<part name="R5" library="rcl" deviceset="R-US_" device="M1206"/>
+<part name="R5" library="rcl" deviceset="R-US_" device="M1206" value="220"/>
 <part name="LED3" library="led" deviceset="LED" device="SMT1206"/>
-<part name="R6" library="rcl" deviceset="R-US_" device="M1206"/>
+<part name="R6" library="rcl" deviceset="R-US_" device="M1206" value="220"/>
 <part name="LED4" library="led" deviceset="LED" device="SMT1206"/>
-<part name="R7" library="rcl" deviceset="R-US_" device="M1206"/>
+<part name="R7" library="rcl" deviceset="R-US_" device="M1206" value="220"/>
 <part name="LED5" library="led" deviceset="LED" device="SMT1206"/>
-<part name="R8" library="rcl" deviceset="R-US_" device="M1206"/>
+<part name="R8" library="rcl" deviceset="R-US_" device="M1206" value="220"/>
 <part name="SMPS" library="pinhead" deviceset="PINHD-1X2" device=""/>
 <part name="VCC_5V" library="SparkFun-Aesthetics" deviceset="VCC" device=""/>
@@
 <part name="GND16" library="SparkFun-Aesthetics" deviceset="GND" device=""/>
 <part name="GND17" library="SparkFun-Aesthetics" deviceset="GND" device=""/>
+<part name="D17" library="diode" deviceset="ZENER-DIODE" device="SOD80C" value="BZV55-C3V3"/>
+<part name="GND18" library="SparkFun-Aesthetics" deviceset="GND" device=""/>
+<part name="J1" library="con-jack" deviceset="DCJ0202" device=""/>
+<part name="IC3" library="linear" deviceset="LM2596S" device=""/>
 </parts>
 <sheets>
@@
 <instance part="IC1" gate="G$1" x="43.18" y="71.12"/>
 <instance part="IC2" gate="G$1" x="43.18" y="22.86"/>
-<instance part="LED1" gate="G$1" x="-53.34" y="60.96"/>
+<instance part="POWER" gate="G$1" x="-53.34" y="60.96"/>
 <instance part="R1" gate="G$1" x="-53.34" y="71.12" rot="R90"/>
 <instance part="S1" gate="1" x="-66.04" y="91.44" rot="R270"/>
@@
 <instance part="R3" gate="G$1" x="320.04" y="71.12"/>
 <instance part="C1" gate="G$1" x="337.82" y="53.34"/>
-<instance part="R4" gate="G$1" x="330.2" y="66.04" rot="R270"/>
 <instance part="RIGHTC" gate="-1" x="2.54" y="73.66"/>
 <instance part="RIGHTC" gate="-2" x="2.54" y="68.58"/>
@@
 <instance part="GND16" gate="1" x="114.3" y="17.78" rot="MR0"/>
 <instance part="GND17" gate="1" x="114.3" y="0" rot="MR0"/>
+<instance part="D17" gate="G$1" x="350.52" y="50.8" rot="R90"/>
+<instance part="GND18" gate="1" x="-73.66" y="35.56"/>
+<instance part="J1" gate="G$1" x="-91.44" y="43.18"/>
+<instance part="IC3" gate="G$1" x="233.68" y="149.86"/>
 </instances>
 <busses>
@@
 </busses>
 <nets>
-<net name="N$3" class="0">
-<segment>
-<pinref part="S1" gate="1" pin="P"/>
-<pinref part="POWERIN" gate="G$1" pin="2"/>
-<wire x1="-78.74" y1="88.9" x2="-71.12" y2="88.9" width="0.1524" layer="91"/>
-<pinref part="CHARGUEIN" gate="G$1" pin="2"/>
-<wire x1="-81.28" y1="63.5" x2="-83.82" y2="63.5" width="0.1524" layer="91"/>
-<wire x1="-83.82" y1="63.5" x2="-83.82" y2="88.9" width="0.1524" layer="91"/>
-<wire x1="-83.82" y1="88.9" x2="-78.74" y2="88.9" width="0.1524" layer="91"/>
-</segment>
-</net>
 <net name="N$23" class="0">
 <segment>
@@
 <net name="N$1" class="0">
 <segment>
-<pinref part="LED1" gate="G$1" pin="A"/>
+<pinref part="POWER" gate="G$1" pin="A"/>
 <pinref part="R1" gate="G$1" pin="1"/>
 <wire x1="-53.34" y1="63.5" x2="-53.34" y2="66.04" width="0.1524" layer="91"/>
@@
 <wire x1="358.14" y1="73.66" x2="297.18" y2="73.66" width="0.1524" layer="91"/>
 <wire x1="297.18" y1="73.66" x2="297.18" y2="58.42" width="0.1524" layer="91"/>
+<junction x="297.18" y="58.42"/>
 </segment>
 </net>
@@
 </segment>
 </net>
-<net name="N$25" class="0">
-<segment>
+<net name="N$28" class="0">
+<segment>
+<pinref part="R3" gate="G$1" pin="2"/>
+<wire x1="325.12" y1="71.12" x2="330.2" y2="71.12" width="0.1524" layer="91"/>
 <pinref part="R2" gate="G$1" pin="2"/>
 <wire x1="330.2" y1="55.88" x2="330.2" y2="58.42" width="0.1524" layer="91"/>
@@
 <wire x1="350.52" y1="35.56" x2="355.6" y2="35.56" width="0.1524" layer="91"/>
 <wire x1="355.6" y1="35.56" x2="355.6" y2="58.42" width="0.1524" layer="91"/>
-<wire x1="355.6" y1="58.42" x2="337.82" y2="58.42" width="0.1524" layer="91"/>
+<wire x1="355.6" y1="58.42" x2="350.52" y2="58.42" width="0.1524" layer="91"/>
 <pinref part="C1" gate="G$1" pin="1"/>
+<wire x1="350.52" y1="58.42" x2="337.82" y2="58.42" width="0.1524" layer="91"/>
 <wire x1="337.82" y1="58.42" x2="330.2" y2="58.42" width="0.1524" layer="91"/>
 <wire x1="337.82" y1="58.42" x2="337.82" y2="55.88" width="0.1524" layer="91"/>
-<pinref part="R4" gate="G$1" pin="2"/>
-<wire x1="330.2" y1="60.96" x2="330.2" y2="58.42" width="0.1524" layer="91"/>
-</segment>
-</net>
-<net name="N$28" class="0">
-<segment>
-<pinref part="R3" gate="G$1" pin="2"/>
-<pinref part="R4" gate="G$1" pin="1"/>
-<wire x1="325.12" y1="71.12" x2="330.2" y2="71.12" width="0.1524" layer="91"/>
+<wire x1="330.2" y1="71.12" x2="330.2" y2="58.42" width="0.1524" layer="91"/>
+<pinref part="D17" gate="G$1" pin="C"/>
+<wire x1="350.52" y1="53.34" x2="350.52" y2="58.42" width="0.1524" layer="91"/>
+<junction x="330.2" y="58.42"/>
+<junction x="337.82" y="58.42"/>
+<junction x="350.52" y="58.42"/>
 </segment>
 </net>
@@
 </segment>
 <segment>
-<pinref part="LED1" gate="G$1" pin="C"/>
+<pinref part="POWER" gate="G$1" pin="C"/>
 <wire x1="-53.34" y1="48.26" x2="-53.34" y2="55.88" width="0.1524" layer="91"/>
 <pinref part="GND6" gate="1" pin="GND"/>
@@
 <wire x1="297.18" y1="45.72" x2="297.18" y2="27.94" width="0.1524" layer="91"/>
 <wire x1="297.18" y1="45.72" x2="330.2" y2="45.72" width="0.1524" layer="91"/>
+<pinref part="D17" gate="G$1" pin="A"/>
+<wire x1="350.52" y1="48.26" x2="350.52" y2="45.72" width="0.1524" layer="91"/>
+<wire x1="350.52" y1="45.72" x2="337.82" y2="45.72" width="0.1524" layer="91"/>
+<junction x="330.2" y="45.72"/>
+<junction x="337.82" y="45.72"/>
 </segment>
 <segment>
@@
 <junction x="386.08" y="25.4"/>
 <junction x="398.78" y="25.4"/>
+<junction x="411.48" y="25.4"/>
+<junction x="373.38" y="25.4"/>
 </segment>
 <segment>
@@
 <pinref part="D14" gate="G$1" pin="A"/>
 <wire x1="114.3" y1="20.32" x2="109.22" y2="20.32" width="0.1524" layer="91"/>
+</segment>
+<segment>
+<pinref part="GND18" gate="1" pin="GND"/>
+<wire x1="-73.66" y1="38.1" x2="-73.66" y2="40.64" width="0.1524" layer="91"/>
+<pinref part="J1" gate="G$1" pin="3"/>
+<wire x1="-73.66" y1="40.64" x2="-83.82" y2="40.64" width="0.1524" layer="91"/>
 </segment>
 </net>
@@
 <wire x1="-30.48" y1="53.34" x2="-30.48" y2="38.1" width="0.1524" layer="91"/>
 <pinref part="R1" gate="G$1" pin="2"/>
-<wire x1="0" y1="81.28" x2="-53.34" y2="76.2" width="0.1524" layer="91"/>
 <wire x1="5.08" y1="81.28" x2="5.08" y2="88.9" width="0.1524" layer="91"/>
 <wire x1="5.08" y1="88.9" x2="20.32" y2="88.9" width="0.1524" layer="91"/>
@@
 <junction x="142.24" y="109.22"/>
 <junction x="147.32" y="109.22"/>
-</segment>
-</net>
+<wire x1="0" y1="81.28" x2="-53.34" y2="81.28" width="0.1524" layer="91"/>
+<wire x1="-53.34" y1="81.28" x2="-53.34" y2="76.2" width="0.1524" layer="91"/>
+</segment>
+</net>
+<net name="N$3" class="0">
+<segment>
+<wire x1="-78.74" y1="45.72" x2="-78.74" y2="50.8" width="0.1524" layer="91"/>
+<wire x1="-78.74" y1="50.8" x2="-93.98" y2="50.8" width="0.1524" layer="91"/>
+<wire x1="-93.98" y1="50.8" x2="-93.98" y2="71.12" width="0.1524" layer="91"/>
+<pinref part="S1" gate="1" pin="P"/>
+<pinref part="POWERIN" gate="G$1" pin="2"/>
+<wire x1="-78.74" y1="88.9" x2="-71.12" y2="88.9" width="0.1524" layer="91"/>
+<pinref part="CHARGUEIN" gate="G$1" pin="2"/>
+<wire x1="-81.28" y1="63.5" x2="-83.82" y2="63.5" width="0.1524" layer="91"/>
+<wire x1="-83.82" y1="63.5" x2="-83.82" y2="71.12" width="0.1524" layer="91"/>
+<wire x1="-83.82" y1="71.12" x2="-83.82" y2="88.9" width="0.1524" layer="91"/>
+<wire x1="-83.82" y1="88.9" x2="-78.74" y2="88.9" width="0.1524" layer="91"/>
+<wire x1="-93.98" y1="71.12" x2="-83.82" y2="71.12" width="0.1524" layer="91"/>
+<pinref part="J1" gate="G$1" pin="1"/>
+<wire x1="-83.82" y1="45.72" x2="-78.74" y2="45.72" width="0.1524" layer="91"/>
+</segment>
+</net>

Commit message: An SMPS and Ref Voltage was added to PiDrive
Parts:
- removed IC3: (no value), linear:LM2596S
- added C2: (no value), rcl:C-EUC1206
- added C3: 100 uF MCGPR25V107M6.3X11, rcl:CPOL-USE1.8-4
- added C4: 68 uF 10MS568MEFC6.3X5, rcl:CPOL-USE1.8-4
- added C5: 10 nF CC1206KRX7R9BB103, rcl:C-EUC1206
- added C6: 0.47 uF C1206C474K5RACTU, rcl:C-EUC1206
- added D18: (no value), diode:DIODE-DO-214AC
- added JP1: (no value), jumper:JP2E
- added L1: 47 uH 13R473C, rcl:L-US6000-XXX-RC
- added U1: LM2675M-5.0, LM2675M-5.0:LM2675M-5.0
- added U2: REF3033AIDBZT, TI-REF3033AIDBZT:REF3033AIDBZT
Connections:
- net RA2 renamed N$15
- removed net N$15 (its old number): R6.2, U$1.RA3/AN3
- removed net RA4: R7.2, U$1.RA4/AN4
- removed net RA5: R8.2, U$1.RA5/MCLR
- new net N$25: C5.2, D18.C, L1.1, U1.VSW
- new net N$27: C3.+, JP1.3, U1.VIN
- new net N$31: R6.2, U$1.RA5/MCLR
- new net N$40: C5.1, U1.CB
- new net N$42: R7.2, U$1.RB0/INT
- new net N$45: C1.2, C2.2, C3.-, C4.-, CHARGUEIN.1, D10.A, D12.A, D14.A, D16.A, D17.A, D18.A, D2.A, D4.A, D6.A, D8.A, IC1.GND1, IC1.GND2, IC1.GND3, IC1.GND4, IC2.GND1, IC2.GND2, IC2.GND3, IC2.GND4, J1.3, LED2.C, LED3.C, LED4.C, LED5.C, MPU6050.2, POWER.C, POWERIN.1, R2.1, SK1.GND@25, SMPS.1, U$1.VSS, U1.GND
- new net N$48: R8.2, U$1.RB1/SDA
- new net N$49: U$1.RA3/AN3, U2.OUT
- net GND: now also C6.1, U2.GND; no longer C1.2, CHARGUEIN.1, D10.A, D12.A, D14.A, D16.A, D17.A, D2.A, D4.A, D6.A, D8.A, IC1.GND1, IC1.GND2, IC1.GND3, IC1.GND4, IC2.GND1, IC2.GND2, IC2.GND3, IC2.GND4, J1.3, LED2.C, LED3.C, LED4.C, LED5.C, MPU6050.2, POWER.C, POWERIN.1, R2.1, SK1.GND@25, SMPS.1, U$1.VSS
- net N$17: now also C2.1
- net N$3: now also JP1.1, JP1.2
- net VCC: now also C4.+, C6.2, L1.2, U1.FB, U2.IN

Commit message: some traces were fixed, the newark bom was added
Parts:
- C1: value 10uF -> 10uF C1206C106K4RACTU
- C2: value (none) -> 10 nF
- C4: value 68 uF 10MS568MEFC6.3X5 -> 68 uF EKZE160ELL680MF07D
- D18: value (none) -> SSA23L-E3/61T
- R1: value 1.5k -> 4k
- R2: value 3.01k -> 422
- R3: value 2k -> 2.61k
Connections:
- removed net N$3: CHARGUEIN.2, J1.1, JP1.1, JP1.2, POWERIN.2, S1.P
- new net N$53: CHARGUEIN.2, J1.1, JP1.1, JP1.2, POWERIN.2, R3.1, S1.P
- net N$10: no longer R3.1
